File: CustomPCBs/ReadyToTest/BNO085_0x4A_Board/BNO085_0x4A_Board.kicad_sch (KiCad schematic)
At the start: 12 parts, among them J1 Conn_01x04_Pin, Y1 32.768kHz

Commit message: Updating IMU boards for different wire connections
Now all components are placed on one layer, making assembly easier. The
JST connector was dropped for smalled IMU housing, instead the wires now
solder directly to the board and exit from the sides of the board.
Parts:
- J1: footprint Connector_JST:JST_SH_SM04B-SRSS-TB_1x04-1MP_P1.00mm_Horizontal -> Library:WireToBoard2x2Wide
Changed lines of the file:
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@@
     (pin "2")
     (instances
-      (project "IMUBoard1QwiicConnector"
+      (project "BNO085_0x4A_Board"
         (path "/70e5a8fd-d79a-42f0-963c-2c04abcfaf88"
           (reference "R4") (unit 1)
@@
     (pin "2")
     (instances
-      (project "IMUBoard1QwiicConnector"
+      (project "BNO085_0x4A_Board"
         (path "/70e5a8fd-d79a-42f0-963c-2c04abcfaf88"
           (reference "R1") (unit 1)
@@
     (pin "2")
     (instances
-      (project "IMUBoard1QwiicConnector"
+      (project "BNO085_0x4A_Board"
         (path "/70e5a8fd-d79a-42f0-963c-2c04abcfaf88"
           (reference "C6") (unit 1)
@@
     (pin "2")
     (instances
-      (project "IMUBoard1QwiicConnector"
+      (project "BNO085_0x4A_Board"
         (path "/70e5a8fd-d79a-42f0-963c-2c04abcfaf88"
           (reference "C1") (unit 1)
@@
     (pin "1")
     (instances
-      (project "IMUBoard1QwiicConnector"
+      (project "BNO085_0x4A_Board"
         (path "/70e5a8fd-d79a-42f0-963c-2c04abcfaf88"
           (reference "#PWR02") (unit 1)
@@
     (pin "1")
     (instances
-      (project "IMUBoard1QwiicConnector"
+      (project "BNO085_0x4A_Board"
         (path "/70e5a8fd-d79a-42f0-963c-2c04abcfaf88"
           (reference "#PWR011") (unit 1)
@@
     (pin "2")
     (instances
-      (project "IMUBoard1QwiicConnector"
+      (project "BNO085_0x4A_Board"
         (path "/70e5a8fd-d79a-42f0-963c-2c04abcfaf88"
           (reference "C5") (unit 1)
@@
       (effects (font (size 1.27 1.27)))
     )
-    (property "Footprint" "Connector_JST:JST_SH_SM04B-SRSS-TB_1x04-1MP_P1.00mm_Horizontal" (at 25.4 38.1 0)
+    (property "Footprint" "Library:WireToBoard2x2Wide" (at 25.4 38.1 0)
       (effects (font (size 1.27 1.27)) hide)
     )
@@
     (pin "4")
     (instances
-      (project "IMUBoard1QwiicConnector"
+      (project "BNO085_0x4A_Board"
         (path "/70e5a8fd-d79a-42f0-963c-2c04abcfaf88"
           (reference "J1") (unit 1)
@@
     (pin "9")
     (instances
-      (project "IMUBoard1QwiicConnector"
+      (project "BNO085_0x4A_Board"
         (path "/70e5a8fd-d79a-42f0-963c-2c04abcfaf88"
           (reference "U1") (unit 1)
@@
     (pin "1")
     (instances
-      (project "IMUBoard1QwiicConnector"
+      (project "BNO085_0x4A_Board"
         (path "/70e5a8fd-d79a-42f0-963c-2c04abcfaf88"
           (reference "#PWR06") (unit 1)
@@
     (pin "1")
     (instances
-      (project "IMUBoard1QwiicConnector"
+      (project "BNO085_0x4A_Board"
         (path "/70e5a8fd-d79a-42f0-963c-2c04abcfaf88"
           (reference "#PWR08") (unit 1)
@@
     (pin "2")
     (instances
-      (project "IMUBoard1QwiicConnector"
+      (project "BNO085_0x4A_Board"
         (path "/70e5a8fd-d79a-42f0-963c-2c04abcfaf88"
           (reference "C4") (unit 1)
@@
     (pin "2")
     (instances
-      (project "IMUBoard1QwiicConnector"
+      (project "BNO085_0x4A_Board"
         (path "/70e5a8fd-d79a-42f0-963c-2c04abcfaf88"
           (reference "Y1") (unit 1)
@@
     (pin "1")
     (instances
-      (project "IMUBoard1QwiicConnector"
+      (project "BNO085_0x4A_Board"
         (path "/70e5a8fd-d79a-42f0-963c-2c04abcfaf88"
           (reference "#PWR03") (unit 1)
@@
     (pin "1")
     (instances
-      (project "IMUBoard1QwiicConnector"
+      (project "BNO085_0x4A_Board"
         (path "/70e5a8fd-d79a-42f0-963c-2c04abcfaf88"
           (reference "#PWR010") (unit 1)
@@
     (pin "2")
     (instances
-      (project "IMUBoard1QwiicConnector"
+      (project "BNO085_0x4A_Board"
         (path "/70e5a8fd-d79a-42f0-963c-2c04abcfaf88"
           (reference "C2") (unit 1)
@@
     (pin "1")
     (instances
-      (project "IMUBoard1QwiicConnector"
+      (project "BNO085_0x4A_Board"
         (path "/70e5a8fd-d79a-42f0-963c-2c04abcfaf88"
           (reference "#PWR01") (unit 1)
@@
     (pin "1")
     (instances
-      (project "IMUBoard1QwiicConnector"
+      (project "BNO085_0x4A_Board"
         (path "/70e5a8fd-d79a-42f0-963c-2c04abcfaf88"
           (reference "#PWR09") (unit 1)
@@
     (pin "2")
     (instances
-      (project "IMUBoard1QwiicConnector"
+      (project "BNO085_0x4A_Board"
         (path "/70e5a8fd-d79a-42f0-963c-2c04abcfaf88"
           (reference "R3") (unit 1)
@@
     (pin "2")
     (instances
-      (project "IMUBoard1QwiicConnector"
+      (project "BNO085_0x4A_Board"
         (path "/70e5a8fd-d79a-42f0-963c-2c04abcfaf88"
           (reference "R2") (unit 1)
@@
     (pin "1")
     (instances
-      (project "IMUBoard1QwiicConnector"
+      (project "BNO085_0x4A_Board"
         (path "/70e5a8fd-d79a-42f0-963c-2c04abcfaf88"
           (reference "#PWR012") (unit 1)
