File: CustomPCBs/InDevelopment/BMI270-and-QMC5883L/BMI270-and-QMC5883L.kicad_sch (KiCad schematic)
At the start: 15 parts, among them J1 Conn_01x04, J2 Conn_01x04, U1 BMI270, U2 QMC5883L

Commit message: Saving work on a new IMU board
Parts:
- removed C1: 100n, Capacitor_SMD:C_0201_0603Metric, symbol Device:C
- removed R3, R4: 2k2, Resistor_SMD:R_0201_0603Metric, symbol Device:R
- C3: footprint Capacitor_SMD:C_0201_0603Metric -> Capacitor_SMD:C_0603_1608Metric; LCSC Part # (none) -> C5252398
- C4: LCSC Part # (none) -> C962109
- R1, R2: value 10k -> 2k2; LCSC Part # C2930027 -> C142018
- U1: LCSC Part # (none) -> C2836813
- U2: LCSC Part # (none) -> C976032
Other:
- moved on the sheet: C2, C3, C4, J2, U2
